File: Double Stack.kicad_pcb (KiCad board)
At the start: 2 copper layers, 54.6 x 52.7 mm, 40 parts, among them J1 Conn_01x06_Male, J2 Barrel_Jack_Switch, Q1 BC547, Q2 BC547, Q3 BC547, Q4 BC547

Commit message: Migrate to KiCAD 6
Parts:
- moved RV1 5.04 mm to (99.7, 60.3)
- moved RV2 5.04 mm to (126.4, 60.3)
Connections:
- J1 pad 2: Net-(J1-Pad2) -> unconnected-(J1-Pad2)
- RV1 pad 1: Net-(C4-Pad1) -> GND
- RV1 pad 3: GND -> Net-(C4-Pad1)
- RV2 pad 1: Net-(C10-Pad1) -> GND
- RV2 pad 3: GND -> Net-(C10-Pad1)
Other:
- net class Default removed
